File: TopPanel.brd (EAGLE design)
At the start: 97.5 x 97.5 mm, 19 parts

Commit message: Connector swap
Parts:
- removed JP5: M02PTH, SparkFun-Connectors:1X02
- added J1: EM406, SparkFun-Connectors:1X06-1MM
Connections:
- net GND: now also J1.1; no longer JP5.1
- net VSOLAR: now also J1.2; no longer JP5.2
Changed lines of the file:
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@@
 <?xml version="1.0" encoding="utf-8"?>
 <!DOCTYPE eagle SYSTEM "eagle.dtd">
-<eagle version="8.6.1">
+<eagle version="9.1.3">
 <drawing>
 <settings>
@@
 <layers>
 <layer number="1" name="Top" color="4" fill="1" visible="yes" active="yes"/>
+<layer number="2" name="Route2" color="1" fill="3" visible="no" active="no"/>
+<layer number="3" name="Route3" color="4" fill="3" visible="no" active="no"/>
+<layer number="4" name="Route4" color="1" fill="4" visible="no" active="no"/>
+<layer number="5" name="Route5" color="4" fill="4" visible="no" active="no"/>
+<layer number="6" name="Route6" color="1" fill="8" visible="no" active="no"/>
+<layer number="7" name="Route7" color="4" fill="8" visible="no" active="no"/>
+<layer number="8" name="Route8" color="1" fill="2" visible="no" active="no"/>
+<layer number="9" name="Route9" color="4" fill="2" visible="no" active="no"/>
+<layer number="10" name="Route10" color="1" fill="7" visible="no" active="no"/>
+<layer number="11" name="Route11" color="4" fill="7" visible="no" active="no"/>
+<layer number="12" name="Route12" color="1" fill="5" visible="no" active="no"/>
+<layer number="13" name="Route13" color="4" fill="5" visible="no" active="no"/>
+<layer number="14" name="Route14" color="1" fill="6" visible="no" active="no"/>
+<layer number="15" name="Route15" color="4" fill="6" visible="no" active="no"/>
 <layer number="16" name="Bottom" color="1" fill="1" visible="yes" active="yes"/>
 <layer number="17" name="Pads" color="2" fill="1" visible="yes" active="yes"/>
@@
 <layer number="54" name="bGND_GNDA" color="1" fill="9" visible="no" active="no"/>
 <layer number="56" name="wert" color="7" fill="1" visible="no" active="no"/>
+<layer number="57" name="tCAD" color="7" fill="1" visible="no" active="no"/>
+<layer number="59" name="tCarbon" color="7" fill="1" visible="no" active="no"/>
+<layer number="60" name="bCarbon" color="7" fill="1" visible="no" active="no"/>
 <layer number="88" name="SimResults" color="9" fill="1" visible="no" active="no"/>
 <layer number="89" name="SimProbes" color="9" fill="1" visible="no" active="no"/>
@@
 <layer number="97" name="Info" color="7" fill="1" visible="no" active="no"/>
 <layer number="98" name="Guide" color="6" fill="1" visible="no" active="no"/>
+<layer number="99" name="SpiceOrder" color="7" fill="1" visible="no" active="no"/>
 <layer number="100" name="Muster" color="7" fill="1" visible="no" active="no"/>
 <layer number="101" name="Patch_Top" color="12" fill="4" visible="yes" active="yes"/>
@@
 <layer number="112" name="tSilk" color="7" fill="1" visible="yes" active="yes"/>
 <layer number="113" name="IDFDebug" color="4" fill="1" visible="yes" active="yes"/>
+<layer number="114" name="Badge_Outline" color="7" fill="1" visible="yes" active="yes"/>
+<layer number="115" name="ReferenceISLANDS" color="7" fill="1" visible="yes" active="yes"/>
 <layer number="116" name="Patch_BOT" color="9" fill="4" visible="yes" active="yes"/>
+<layer number="118" name="Rect_Pads" color="7" fill="1" visible="yes" active="yes"/>
 <layer number="121" name="_tsilk" color="7" fill="1" visible="yes" active="yes"/>
 <layer number="122" name="_bsilk" color="7" fill="1" visible="yes" active="yes"/>
@@
 <layer number="127" name="_tValues" color="7" fill="1" visible="yes" active="yes"/>
 <layer number="128" name="_bValues" color="7" fill="1" visible="yes" active="yes"/>
+<layer number="129" name="Mask" color="7" fill="1" visible="yes" active="yes"/>
 <layer number="131" name="tAdjust" color="7" fill="1" visible="yes" active="yes"/>
 <layer number="132" name="bAdjust" color="7" fill="1" visible="yes" active="yes"/>
 <layer number="144" name="Drill_legend" color="7" fill="1" visible="yes" active="yes"/>
+<layer number="150" name="Notes" color="7" fill="1" visible="yes" active="yes"/>
 <layer number="151" name="HeatSink" color="7" fill="1" visible="yes" active="yes"/>
 <layer number="152" name="_bDocu" color="7" fill="1" visible="yes" active="yes"/>
+<layer number="153" name="FabDoc1" color="7" fill="1" visible="yes" active="yes"/>
+<layer number="154" name="FabDoc2" color="7" fill="1" visible="yes" active="yes"/>
+<layer number="155" name="FabDoc3" color="7" fill="1" visible="yes" active="yes"/>
 <layer number="199" name="Contour" color="7" fill="1" visible="yes" active="yes"/>
 <layer number="200" name="200bmp" color="1" fill="10" visible="yes" active="yes"/>
@@
 <layer number="223" name="223bmp" color="24" fill="1" visible="no" active="no"/>
 <layer number="224" name="224bmp" color="25" fill="1" visible="no" active="no"/>
+<layer number="225" name="225bmp" color="7" fill="1" visible="yes" active="yes"/>
+<layer number="226" name="226bmp" color="7" fill="1" visible="yes" active="yes"/>
+<layer number="227" name="227bmp" color="7" fill="1" visible="yes" active="yes"/>
+<layer number="228" name="228bmp" color="7" fill="1" visible="yes" active="yes"/>
+<layer number="229" name="229bmp" color="7" fill="1" visible="yes" active="yes"/>
+<layer number="230" name="230bmp" color="7" fill="1" visible="yes" active="yes"/>
+<layer number="231" name="231bmp" color="7" fill="1" visible="yes" active="yes"/>
+<layer number="232" name="Eagle3D_PG2" color="7" fill="1" visible="yes" active="yes"/>
+<layer number="233" name="Eagle3D_PG3" color="7" fill="1" visible="yes" active="yes"/>
 <layer number="248" name="Housing" color="7" fill="1" visible="yes" active="yes"/>
 <layer number="249" name="Edge" color="7" fill="1" visible="yes" active="yes"/>
@@
 <layer number="251" name="SMDround" color="12" fill="11" visible="no" active="no"/>
 <layer number="254" name="cooling" color="7" fill="1" visible="yes" active="yes"/>
+<layer number="255" name="routoute" color="7" fill="1" visible="yes" active="yes"/>
 </layers>
 <board>
@@
 <param name="checkStop" value="0"/>
 <param name="checkValues" value="0"/>
+<param name="checkNames" value="1"/>
+<param name="checkWireStubs" value="1"/>
+<param name="checkPolygonWidth" value="0"/>
 <param name="useDiameter" value="13"/>
 <param name="maxErrors" value="50"/>
@@
 <element name="D6" library="Solar" package="SB_DIODE" value="SB_DIODE" x="55.2" y="-96.6"/>
 <element name="FRAME1" library="SparkFun-Aesthetics" package="CREATIVE_COMMONS" value="FRAME-LETTER" x="21" y="-92.5"/>
-<element name="JP5" library="SparkFun-Connectors" package="1X02" value="M02PTH" x="9.4" y="-75.4"/>
 <element name="U$1" library="KickSat-Logo" package="KICKSAT_LOGO" value="KICKSAT_LOGO" x="22.4" y="-76.8"/>
+<element name="J1" library="SparkFun-Connectors" library_urn="urn:adsk.eagle:library:513" package="1X06-1MM" package3d_urn="urn:adsk.eagle:package:38023/1" value="EM406" x="12" y="12" rot="MR45">
+<attribute name="PROD_ID" value="CONN-08249" x="12" y="12" size="1.778" layer="28" rot="MR45" display="off"/>
+<attribute name="SF_ID" value="GPS-00579" x="12" y="12" size="1.778" layer="28" rot="MR45" display="off"/>
+</element>
 </elements>
 <signals>
@@
 <signal name="VSOLAR">
 <contactref element="D6" pad="NEG"/>
-<contactref element="JP5" pad="2"/>
-<wire x1="54" y1="-96.6" x2="11.94" y2="-75.4" width="0" layer="19" extent="1-1"/>
+<contactref element="J1" pad="2"/>
+<wire x1="13.986971875" y1="11.809078125" x2="54" y2="-96.6" width="0" layer="19" extent="1-16"/>
 </signal>
 <signal name="N$37">
@@
 <contactref element="D5" pad="POS"/>
 <contactref element="SL10" pad="1"/>
-<contactref element="JP5" pad="1"/>
 <polygon width="0.1524" layer="16">
 <vertex x="0" y="8"/>
@@
 <vertex x="0" y="89.5"/>
 </polygon>
-<wire x1="47.15" y1="-96.6" x2="9.4" y2="-75.4" width="0" layer="19" extent="1-1"/>
-<wire x1="45.5107" y1="-38.7009" x2="9.4" y2="-75.4" width="0" layer="19" extent="1-1"/>
+<contactref element="J1" pad="1"/>
+<wire x1="45.5107" y1="-38.7009" x2="47.15" y2="-96.6" width="0" layer="19" extent="1-1"/>
 <wire x1="60.4107" y1="-38.7009" x2="45.5107" y2="-38.7009" width="0" layer="19" extent="1-1"/>
+<wire x1="14.694078125" y1="11.101971875" x2="45.5107" y2="-38.7009" width="0" layer="19" extent="1-16"/>
 </signal>
 </signals>
+<mfgpreviewcolors>
+<mfgpreviewcolor name="soldermaskcolor" color="0xC8008000"/>
+<mfgpreviewcolor name="silkscreencolor" color="0xFFFEFEFE"/>
+<mfgpreviewcolor name="backgroundcolor" color="0xFF282828"/>
+<mfgpreviewcolor name="coppercolor" color="0xFFFFBF00"/>
+<mfgpreviewcolor name="substratecolor" color="0xFF786E46"/>
+</mfgpreviewcolors>
 </board>
 </drawing>
+<compatibility>
+<note version="8.2" severity="warning">
+Since Version 8.2, EAGLE supports online libraries. The ids
+of those online libraries will not be understood (or retained)
+with this version.
+</note>
+<note version="8.3" severity="warning">
+Since Version 8.3, EAGLE supports URNs for individual library
+assets (packages, symbols, and devices). The URNs of those assets
+will not be understood (or retained) with this version.
+</note>
+<note version="8.3" severity="warning">
+Since Version 8.3, EAGLE supports the association of 3D packages
+with devices in libraries, schematics, and board files. Those 3D
+packages will not be understood (or retained) with this version.
+</note>
+</compatibility>
 </eagle>

Commit message: put connector in correct spot
Parts:
- moved J1 5.66 mm to (16.0, 16.0), turned to 225 degrees
Changed lines of the file:
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@@
 <wire x1="60.340428125" y1="58.93621875" x2="58.92621875" y2="60.350428125" width="0.1" layer="20"/>
 <wire x1="58.92621875" y1="60.350428125" x2="58.92621875" y2="64.593071875" width="0.1" layer="20" curve="-90"/>
+<circle x="14.75" y="14.75" radius="4.25" width="0.254" layer="21"/>
 </plain>
 <attributes>
@@
 <element name="FRAME1" library="SparkFun-Aesthetics" package="CREATIVE_COMMONS" value="FRAME-LETTER" x="21" y="-92.5"/>
 <element name="U$1" library="KickSat-Logo" package="KICKSAT_LOGO" value="KICKSAT_LOGO" x="22.4" y="-76.8"/>
-<element name="J1" library="SparkFun-Connectors" library_urn="urn:adsk.eagle:library:513" package="1X06-1MM" package3d_urn="urn:adsk.eagle:package:38023/1" value="EM406" x="12" y="12" rot="MR45">
-<attribute name="PROD_ID" value="CONN-08249" x="12" y="12" size="1.778" layer="28" rot="MR45" display="off"/>
-<attribute name="SF_ID" value="GPS-00579" x="12" y="12" size="1.778" layer="28" rot="MR45" display="off"/>
+<element name="J1" library="SparkFun-Connectors" library_urn="urn:adsk.eagle:library:513" package="1X06-1MM" package3d_urn="urn:adsk.eagle:package:38023/1" value="EM406" x="16" y="16" rot="MR225">
+<attribute name="PROD_ID" value="CONN-08249" x="16" y="16" size="1.778" layer="28" rot="MR225" display="off"/>
+<attribute name="SF_ID" value="GPS-00579" x="16" y="16" size="1.778" layer="28" rot="MR225" display="off"/>
 </element>
 </elements>
@@
 <contactref element="D6" pad="NEG"/>
 <contactref element="J1" pad="2"/>
-<wire x1="13.986971875" y1="11.809078125" x2="54" y2="-96.6" width="0" layer="19" extent="1-16"/>
+<wire x1="14.01303125" y1="16.19091875" x2="54" y2="-96.6" width="0" layer="19" extent="1-16"/>
 </signal>
 <signal name="N$37">
@@
 <wire x1="45.5107" y1="-38.7009" x2="47.15" y2="-96.6" width="0" layer="19" extent="1-1"/>
 <wire x1="60.4107" y1="-38.7009" x2="45.5107" y2="-38.7009" width="0" layer="19" extent="1-1"/>
-<wire x1="14.694078125" y1="11.101971875" x2="45.5107" y2="-38.7009" width="0" layer="19" extent="1-16"/>
+<wire x1="13.305925" y1="16.898025" x2="45.5107" y2="-38.7009" width="0" layer="19" extent="1-16"/>
 </signal>
 </signals>

Commit message: Started routing
Parts:
- added U$2, U$3, U$4: BURNWIRE, BurnWire:BURNWIRE
- moved D3 170.0 mm to (6.70, 72.4)
- moved D4 169.5 mm to (49.0, 72.4)
- moved D5 169.2 mm to (65.9, 71.3), turned to 180 degrees
- moved SL10 134.8 mm to (79.0, 92.0), turned to 270 degrees
- moved SL8 133.7 mm to (35.0, 92.0), turned to 270 degrees
- moved D2 121.1 mm to (30.5, 23.6)
- moved D1 118.1 mm to (57.1, 9.70)
- moved SL9 117.6 mm to (62.0, 75.0), turned to 90 degrees
- moved SL7 116.7 mm to (18.0, 75.0), turned to 90 degrees
- moved D6 110.3 mm to (14.2, 5.80), turned to 270 degrees
- moved SL6 83.7 mm to (36.0, 35.0), turned to 180 degrees
- moved SL5 78.3 mm to (21.0, 58.0)
- moved SL3 70.4 mm to (83.0, 40.0), turned to 270 degrees
- moved SL2 65.8 mm to (76.0, 21.0), turned to 270 degrees
- moved SL4 36.6 mm to (55.0, 27.0), turned to 90 degrees
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Connections:
- new net VBURN1: J1.2, U$2.V+
- new net VBURN2: J1.3, U$3.V+
- new net VBURN3: J1.4, U$4.V+
- net GND: now also J1.5, U$2.V-, U$3.V-, U$4.V-
- net VSOLAR: now also J1.6; no longer J1.2
Routing:
- net VBURN1: track 0.00 -> 60.4 mm, vias 0 -> 1
- net VBURN2: track 0.00 -> 56.7 mm, vias 0 -> 1
- net VBURN3: track 0.00 -> 55.7 mm, vias 0 -> 1
- net N$50: track 0.00 -> 48.3 mm
- net GND: track 0.00 -> 17.5 mm, vias 0 -> 5

Commit message: Finished layout
Parts:
- moved U$1 133.1 mm to (3.10, 54.9), turned to 270 degrees
- moved FRAME1 130.9 mm to (70.7, 28.6), flipped to the bottom
- moved D1 26.0 mm to (32.9, 19.1), turned to 90 degrees
- moved D3 14.8 mm to (21.3, 70.2), turned to 180 degrees
- moved D2 12.5 mm to (42.8, 25.7), turned to 90 degrees
- moved D6 1.92 mm to (13.3, 7.50)
- moved D4 0.81 mm to (48.2, 72.3)
Routing:
- net N$45: track 0.00 -> 166.2 mm
- net N$39: track 0.00 -> 141.4 mm
- net N$37: track 0.00 -> 120.1 mm
- net N$50: track 48.3 -> 142.4 mm
- net N$9: track 0.00 -> 73.2 mm
- net VSOLAR: track 0.00 -> 6.18 mm, vias 0 -> 1
